File: cmsis-dap_rp2040/cmsis-dap_rp2040.kicad_pcb (KiCad board)
At the start: 2 copper layers, 50 x 34 mm, 61 parts, among them J1 USB_C_Receptacle_USB2.0, J2 UART, J3 RP2040_SWD, J4 Conn_ARM_JTAG_SWD_20, SW1 BOOT, SW2 RUN, U1 SIT2001B, U2 W25Q16JVSSIM, U3 RP2040, U4 NCP1117ST33T3G

Commit message: Release v2022.06.01
Parts:
- removed J3: RP2040_SWD, Connector_PinHeader_2.54mm:PinHeader_1x03_P2.54mm_Vertical
- removed SW1: BOOT, Button_Switch_SMD:SW_Push_SPST_NO_Alps_SKRK
- removed SW2: RUN, Button_Switch_SMD:SW_Push_SPST_NO_Alps_SKRK
- removed TP4: HandSolderHole, TestPoint:TestPoint_THTPad_2.0x2.0mm_Drill1.0mm
- added TP10: TestPoint, TestPoint:TestPoint_Pad_D1.0mm, B.Cu at (103.7, 58.8)
- added TP8: TestPoint, TestPoint:TestPoint_Pad_D1.0mm, B.Cu at (115.8, 59.3)
- added TP9: TestPoint, TestPoint:TestPoint_Pad_D1.0mm, B.Cu at (117.6, 58.4)
- C11, C13, C15, C17, C18, C5, C6, C8, C9: moved to F.Cu
- C7, R2, R8: moved to B.Cu
- J2: value UART -> BOOT; footprint Connector_PinHeader_2.54mm:PinHeader_1x04_P2.54mm_Vertical -> Connector_PinHeader_2.54mm:PinHeader_1x02_P2.54mm_Vertical
- L1: value 600R/0.5A/N.F. -> N.F.
- L2: value 600R/0.5A -> N.F.
- U3: footprint Package_DFN_QFN:QFN-56-1EP_7x7mm_P0.4mm_EP5.6x5.6mm -> rp2040:RP2040_QFN56_HandSolderHack
- moved R8 7.76 mm to (127.9, 68.8), turned to 90 degrees
- moved R12 7.17 mm to (124.1, 64.8), turned to 180 degrees
- moved R1 6.45 mm to (122.4, 59.2), turned to 90 degrees
- moved R2 6.40 mm to (118.8, 53.2), turned to 270 degrees
- moved R9 5.56 mm to (119.6, 58.8), turned to 90 degrees
- moved C8 5.04 mm to (115.0, 64.7), turned to 270 degrees
- moved C7 4.88 mm to (126.4, 68.8), turned to 270 degrees
- moved C2 4.48 mm to (124.9, 59.6), turned to 180 degrees
- moved R10 3.50 mm to (128.1, 77.0), turned to 0 degrees
- moved R13 3.42 mm to (122.5, 71.9)
- moved R16 3.41 mm to (121.1, 58.8), turned to 90 degrees
- moved J2 3.21 mm to (124.0, 52.4), turned to 270 degrees
- moved C9 3.17 mm to (113.5, 64.7), turned to 270 degrees
- moved D4 3.07 mm to (131.1, 77.0), turned to 180 degrees
- moved C13 2.98 mm to (122.5, 67.3), turned to 180 degrees
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Connections:
- net /RUN renamed Net-(C7-Pad1)
- J2 pad 1: +3V3 -> GND
- J2 pad 2: /UART_RX -> /QSPI_CSN
- J4 pad 11: Net-(J4-Pad11) -> (no net)
- R12 pad 1: /RTCK -> Net-(R12-Pad1)
- R12 pad 2: Net-(J4-Pad11) -> /XIN
- R7 pad 1: +3V3 -> /VO
- U1 pad 5: /XIN -> Net-(R12-Pad1)
- U3 pad 24: /SWCLK -> (no net)
- U3 pad 25: /SWDIO -> (no net)
- U3 pad 30: /RTCK -> /TDO_SWO
- U3 pad 31: /TDO_SWO -> /~SRST
- U3 pad 32: /~SRST -> (no net)
Routing:
- net GND: track 122.5 -> 326.3 mm, vias 169 -> 156
- net +3V3: track 144.2 -> 98.4 mm, vias 10 -> 12
- net /SWCLK: track 15.2 -> 0.00 mm
- net Net-(J4-Pad11): track 12.7 -> 0.00 mm
- net +1V1: track 54.1 -> 65.6 mm
- net /UART_TX: track 15.0 -> 4.04 mm
- net /UART_RX: track 12.9 -> 2.89 mm
- net Net-(J4-Pad3): track 12.9 -> 22.6 mm
- net /SWDIO: track 9.63 -> 0.00 mm
- net /LED: track 24.4 -> 16.8 mm
- net Net-(J4-Pad5): track 13.2 -> 20.1 mm
- net /RTCK: track 6.66 -> 0.00 mm
- net /~TRST: track 8.15 -> 2.49 mm
- net /TDI: track 6.55 -> 2.21 mm
- net Net-(J4-Pad7): track 13.5 -> 17.1 mm
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- added copper zone on F.Cu, net /D+
- added copper zone on F.Cu, net /D-
- added copper zone on B.Cu, net /QSPI_CSN
- removed copper zone on F.Cu, net +3V3
- removed copper zone on F.Cu, net /VBUS
Other:
- board text added: "RP2040 CMSIS-DAP version 2022/06/01 @tnishinaga"
- board text removed: "3v3"
- board text removed: "BOOT"
- board text removed: "CLK"
- board text removed: "DIO"
- board text removed: "G"
- board text removed: "GND"
- board text removed: "RP2040 CMSIS-DAP version 2022/04/09 @tnishinaga"
- board text removed: "RUN"
- board text removed: "RX<"
- board text removed: "SWD"
- board text removed: "TX>"
