File: cmsis-dap_rp2040/cmsis-dap_rp2040.sch (KiCad schematic (older format))
At the start: 61 parts, among them J1 USB_C_Receptacle_USB2.0, J2 UART, J3 RP2040_SWD, J4 Conn_ARM_JTAG_SWD_20, SW1 BOOT, SW2 RUN, U1 SIT2001B, U2 W25Q16JVSSIM, U3 RP2040, U4 NCP1117ST33T3G

Commit message: Release v2022.06.01
Parts:
- removed J2: UART, Connector_PinHeader_2.54mm:PinHeader_1x04_P2.54mm_Vertical, symbol Connector:Conn_01x04_Male
- removed J3: RP2040_SWD, Connector_PinHeader_2.54mm:PinHeader_1x03_P2.54mm_Vertical, symbol Connector:Conn_01x03_Male
- removed SW1: BOOT, Button_Switch_SMD:SW_Push_SPST_NO_Alps_SKRK, symbol Switch:SW_Push
- removed SW2: RUN, Button_Switch_SMD:SW_Push_SPST_NO_Alps_SKRK, symbol Switch:SW_Push
- removed TP4: HandSolderHole, TestPoint:TestPoint_THTPad_2.0x2.0mm_Drill1.0mm, symbol Connector:TestPoint
- added J2: BOOT, Connector_PinHeader_2.54mm:PinHeader_1x02_P2.54mm_Vertical, symbol Connector:Conn_01x02_Male
- added TP10, TP8, TP9: TestPoint, TestPoint:TestPoint_Pad_D1.0mm, symbol Connector:TestPoint
- L1: value 600R/0.5A/N.F. -> N.F.
- L2: value 600R/0.5A -> N.F.
- U3: footprint Package_DFN_QFN:QFN-56-1EP_7x7mm_P0.4mm_EP5.6x5.6mm -> rp2040:RP2040_QFN56_HandSolderHack
Connections:
- net +3V3: no longer R7.1
- net GND: now also J2.1 (Pin_1), TP10.1
- net QSPI_CSN: now also J2.2 (Pin_2)
- net TDO_SWO: now also U3.30 (GPIO19); no longer U3.31 (GPIO20)
- net UART_RX: now also TP8.1
- net UART_TX: now also TP9.1
- net VO: now also R7.1
- net XIN: now also R12.2; no longer U1.5 (OUT)
- net ~SRST: now also U3.31 (GPIO20); no longer U3.32 (GPIO21)
- net at J4.11 (RTCK): no longer R12.2
- net RTCK: no longer names the net of R12.1
- net RTCK: now also U1.5 (OUT); no longer U3.30 (GPIO19)
- net RUN: no longer names the net of C7.1, R8.2, U3.26 (RUN)
- net SWCLK: no longer names the net of U3.24 (SWCLK)
- net SWDIO: no longer names the net of U3.25 (SWDIO)
- no-connect marks 27 -> 31
Other:
- note added: "BOOT SELECT"
- note removed: "HandSolderHack"
