File: cmsis-dap_rp2040/panelized/cmsis-dap_rp2040.kicad_pcb (KiCad board)
At the start: 2 copper layers, 103.1 x 81.2 mm, 246 parts, among them J1 USB_C_Receptacle_USB2.0, J2 UART, J3 RP2040_SWD, J4 Conn_ARM_JTAG_SWD_20, SW1 BOOT, SW2 RUN, U1 SIT2001B, U2 W25Q16JVSSIM, U3 RP2040, U4 NCP1117ST33T3G

Commit message: Release v2022.06.01
Parts:
- removed the C11 at (165.8, 105.8)
- removed the C11 at (115.8, 105.8)
- removed the C11 at (165.8, 71.8)
- removed the C12 at (160.3, 102.9)
- removed the C12 at (110.3, 102.9)
- removed the C12 at (160.3, 68.9)
- removed the C12 at (110.3, 68.9)
- removed the C13 at (174.9, 99.6)
- removed the C13 at (124.9, 99.6)
- removed the C13 at (174.9, 65.6)
- removed the C13 at (124.9, 65.6)
- removed the C14 at (174.9, 101.2)
- removed the C14 at (124.9, 101.2)
- removed the C14 at (174.9, 67.2)
- removed the C14 at (124.9, 67.2)
- removed the C15 at (168.8, 105.8)
- removed the C15 at (118.8, 105.8)
- removed the C15 at (168.8, 71.8)
- removed the C15 at (118.8, 71.8)
- removed the C16 at (160.3, 95.2)
- removed the C16 at (110.3, 95.2)
- removed the C16 at (160.3, 61.2)
- removed the C16 at (110.3, 61.2)
- removed the C17 at (169.3, 93.3)
- removed the C17 at (119.3, 93.3)
- removed the C17 at (169.3, 59.3)
- removed the C17 at (119.3, 59.3)
- removed the C18 at (166.0, 93.4)
- removed the C18 at (116.0, 93.4)
- removed the C18 at (166.0, 59.4)
- removed the C18 at (116.0, 59.4)
- removed the C2 at (177.5, 97.3)
- removed the C2 at (127.5, 97.3)
- removed the C2 at (177.5, 63.3)
- removed the C5 at (160.4, 104.4)
- removed the C5 at (110.4, 104.4)
- removed the C5 at (160.4, 70.4)
- removed the C5 at (110.4, 70.4)
- removed the C6 at (164.2, 105.8)
- removed the C6 at (114.2, 105.8)
- removed the C6 at (164.2, 71.8)
- removed the C7 at (171.9, 100.8)
- removed the C7 at (121.9, 100.8)
- removed the C7 at (171.9, 66.8)
- removed the C7 at (121.9, 66.8)
- removed the C8 at (160.3, 96.8)
- removed the C8 at (110.3, 96.8)
- removed the C8 at (160.3, 62.8)
- removed the C9 at (160.3, 98.3)
- removed the C9 at (110.3, 98.3)
- removed the C9 at (160.3, 64.3)
- removed the D3 at (180.0, 114.1)
- removed the D3 at (130.0, 114.1)
- removed the D3 at (180.0, 80.1)
- removed the D4 at (181.5, 114.1)
- removed the D4 at (131.5, 114.1)
- removed the D4 at (181.5, 80.1)
- removed the J2 at (170.8, 86.7)
- removed the J2 at (120.8, 86.7)
- removed the J2 at (170.8, 52.7)
- removed the J2 at (120.8, 52.7)
- removed J3 (x4): RP2040_SWD, Connector_PinHeader_2.54mm:PinHeader_1x03_P2.54mm_Vertical
- removed the R1 at (177.5, 97.3)
- removed the R1 at (127.5, 97.3)
- removed the R1 at (177.5, 63.3)
- removed the R10 at (181.6, 111.0)
- removed the R10 at (131.6, 111.0)
- removed the R10 at (181.6, 77.0)
- removed the R11 at (175.2, 110.0)
- removed the R11 at (125.2, 110.0)
- removed the R11 at (175.2, 76.0)
- removed the R12 at (175.2, 105.8)
- removed the R12 at (125.2, 105.8)
- removed the R12 at (175.2, 71.8)
- removed the R12 at (125.2, 71.8)
- removed the R13 at (175.2, 103.9)
- removed the R13 at (125.2, 103.9)
- removed the R13 at (175.2, 69.9)
- removed the R13 at (125.2, 69.9)
- removed the R14 at (174.4, 93.8)
- removed the R14 at (124.4, 93.8)
- removed the R14 at (174.4, 59.8)
- removed the R15 at (175.2, 107.9)
- removed the R15 at (125.2, 107.9)
- removed the R15 at (175.2, 73.9)
- removed the R16 at (174.4, 91.8)
- removed the R16 at (124.4, 91.8)
- removed the R16 at (174.4, 57.8)
- removed the R2 at (162.4, 87.1)
- removed the R2 at (112.4, 87.1)
- removed the R2 at (162.4, 53.1)
- removed the R3 at (157.4, 97.6)
- removed the R3 at (107.5, 97.6)
- removed the R3 at (157.4, 63.6)
- removed the R5 at (160.3, 101.3)
- removed the R5 at (110.3, 101.3)
- removed the R5 at (160.3, 67.3)
- removed the R6 at (160.3, 99.8)
- removed the R6 at (110.3, 99.8)
- removed the R6 at (160.3, 65.8)
- removed the R7 at (180.0, 111.0)
- removed the R7 at (130.0, 111.0)
- removed the R7 at (180.0, 77.0)
- removed the R8 at (170.4, 100.8)
- removed the R8 at (120.4, 100.8)
- removed the R8 at (170.4, 66.8)
- removed the R8 at (120.4, 66.8)
- removed the R9 at (174.4, 90.0)
- removed the R9 at (124.4, 90.0)
- removed the R9 at (174.4, 56.0)
- removed REF** (x2): TestPoint_Pad_D2.0mm, TestPoint:TestPoint_Pad_D2.0mm
- removed SW1 (x4): BOOT, Button_Switch_SMD:SW_Push_SPST_NO_Alps_SKRK
- removed SW2 (x4): RUN, Button_Switch_SMD:SW_Push_SPST_NO_Alps_SKRK
- removed TP4 (x4): HandSolderHole, TestPoint:TestPoint_THTPad_2.0x2.0mm_Drill1.0mm
- removed the U1 at (174.9, 97.0)
- removed the U1 at (124.9, 97.0)
- removed the U1 at (174.9, 63.0)
- removed the U1 at (124.9, 63.0)
- removed the U3 at (168.4, 99.4)
- removed the U3 at (118.4, 99.4)
- removed the U3 at (168.4, 65.4)
- added C11: 0.1uF, Capacitor_SMD:C_0603_1608Metric, F.Cu at (166.1, 103.8)
- added C11: 0.1uF, Capacitor_SMD:C_0603_1608Metric, F.Cu at (116.1, 103.8)
- added C11: 0.1uF, Capacitor_SMD:C_0603_1608Metric, F.Cu at (166.1, 69.8)
- added C12: 1uF, Capacitor_SMD:C_0603_1608Metric, B.Cu at (161.2, 103.1)
- added C12: 1uF, Capacitor_SMD:C_0603_1608Metric, B.Cu at (111.2, 103.1)
- added C12: 1uF, Capacitor_SMD:C_0603_1608Metric, B.Cu at (161.2, 69.1)
- added C12: 1uF, Capacitor_SMD:C_0603_1608Metric, B.Cu at (111.2, 69.1)
- added C13: 0.1uF, Capacitor_SMD:C_0603_1608Metric, F.Cu at (172.4, 101.3)
- added C13: 0.1uF, Capacitor_SMD:C_0603_1608Metric, F.Cu at (122.5, 101.3)
- added C13: 0.1uF, Capacitor_SMD:C_0603_1608Metric, F.Cu at (172.4, 67.3)
- added C13: 0.1uF, Capacitor_SMD:C_0603_1608Metric, F.Cu at (122.5, 67.3)
- added C14: 0.1uF, Capacitor_SMD:C_0603_1608Metric, B.Cu at (174.9, 101.2)
- added C14: 0.1uF, Capacitor_SMD:C_0603_1608Metric, B.Cu at (124.9, 101.2)
- added C14: 0.1uF, Capacitor_SMD:C_0603_1608Metric, B.Cu at (174.9, 67.2)
- added C14: 0.1uF, Capacitor_SMD:C_0603_1608Metric, B.Cu at (124.9, 67.2)
- added C15: 0.1uF, Capacitor_SMD:C_0603_1608Metric, F.Cu at (168.1, 103.8)
- added C15: 0.1uF, Capacitor_SMD:C_0603_1608Metric, F.Cu at (118.1, 103.8)
- added C15: 0.1uF, Capacitor_SMD:C_0603_1608Metric, F.Cu at (168.1, 69.8)
- added C15: 0.1uF, Capacitor_SMD:C_0603_1608Metric, F.Cu at (118.1, 69.8)
- added C16: 0.1uF, Capacitor_SMD:C_0603_1608Metric, B.Cu at (160.9, 96.6)
- added C16: 0.1uF, Capacitor_SMD:C_0603_1608Metric, B.Cu at (110.9, 96.6)
- added C16: 0.1uF, Capacitor_SMD:C_0603_1608Metric, B.Cu at (160.9, 62.6)
- added C16: 0.1uF, Capacitor_SMD:C_0603_1608Metric, B.Cu at (110.9, 62.6)
- added C17: 0.1uF, Capacitor_SMD:C_0603_1608Metric, F.Cu at (169.1, 95.5)
- added C17: 0.1uF, Capacitor_SMD:C_0603_1608Metric, F.Cu at (119.1, 95.5)
- added C17: 0.1uF, Capacitor_SMD:C_0603_1608Metric, F.Cu at (169.1, 61.5)
- added C17: 0.1uF, Capacitor_SMD:C_0603_1608Metric, F.Cu at (119.1, 61.5)
- added C18: 0.1uF, Capacitor_SMD:C_0603_1608Metric, F.Cu at (166.9, 95.5)
- added C18: 0.1uF, Capacitor_SMD:C_0603_1608Metric, F.Cu at (116.9, 95.5)
- added C18: 0.1uF, Capacitor_SMD:C_0603_1608Metric, F.Cu at (166.9, 61.5)
- added C18: 0.1uF, Capacitor_SMD:C_0603_1608Metric, F.Cu at (116.9, 61.5)
- added C2: 0.1uF, Capacitor_SMD:C_0603_1608Metric, B.Cu at (174.9, 93.6)
- added C2: 0.1uF, Capacitor_SMD:C_0603_1608Metric, B.Cu at (124.9, 93.6)
- added C2: 0.1uF, Capacitor_SMD:C_0603_1608Metric, B.Cu at (174.9, 59.6)
- added C5: 1uF, Capacitor_SMD:C_0603_1608Metric, F.Cu at (162.0, 103.8)
- added C5: 1uF, Capacitor_SMD:C_0603_1608Metric, F.Cu at (112.0, 103.8)
- added C5: 1uF, Capacitor_SMD:C_0603_1608Metric, F.Cu at (162.0, 69.8)
- added C5: 1uF, Capacitor_SMD:C_0603_1608Metric, F.Cu at (112.0, 69.8)
- added C6: 0.1uF, Capacitor_SMD:C_0603_1608Metric, F.Cu at (164.1, 103.8)
- added C6: 0.1uF, Capacitor_SMD:C_0603_1608Metric, F.Cu at (114.1, 103.8)
- added C6: 0.1uF, Capacitor_SMD:C_0603_1608Metric, F.Cu at (164.1, 69.8)
- added C7: 0.1uF, Capacitor_SMD:C_0603_1608Metric, B.Cu at (176.4, 102.8)
- added C7: 0.1uF, Capacitor_SMD:C_0603_1608Metric, B.Cu at (126.4, 102.8)
- added C7: 0.1uF, Capacitor_SMD:C_0603_1608Metric, B.Cu at (176.4, 68.8)
- added C7: 0.1uF, Capacitor_SMD:C_0603_1608Metric, B.Cu at (126.4, 68.8)
- added C8: 0.1uF, Capacitor_SMD:C_0603_1608Metric, F.Cu at (165.0, 98.7)
- added C8: 0.1uF, Capacitor_SMD:C_0603_1608Metric, F.Cu at (115.0, 98.7)
- added C8: 0.1uF, Capacitor_SMD:C_0603_1608Metric, F.Cu at (165.0, 64.7)
- added C9: 0.1uF, Capacitor_SMD:C_0603_1608Metric, F.Cu at (163.5, 98.7)
- added C9: 0.1uF, Capacitor_SMD:C_0603_1608Metric, F.Cu at (113.5, 98.7)
- added C9: 0.1uF, Capacitor_SMD:C_0603_1608Metric, F.Cu at (163.5, 64.7)
- added D3: RED, Diode_SMD:D_0603_1608Metric, F.Cu at (181.1, 112.5)
- added D3: RED, Diode_SMD:D_0603_1608Metric, F.Cu at (131.1, 112.5)
- added D3: RED, Diode_SMD:D_0603_1608Metric, F.Cu at (181.1, 78.5)
- added D4: GREEN, Diode_SMD:D_0603_1608Metric, F.Cu at (181.1, 111.0)
- added D4: GREEN, Diode_SMD:D_0603_1608Metric, F.Cu at (131.1, 111.0)
- added D4: GREEN, Diode_SMD:D_0603_1608Metric, F.Cu at (181.1, 77.0)
- added J2: BOOT, Connector_PinHeader_2.54mm:PinHeader_1x02_P2.54mm_Vertical, F.Cu at (174.0, 86.3)
- added J2: BOOT, Connector_PinHeader_2.54mm:PinHeader_1x02_P2.54mm_Vertical, F.Cu at (124.0, 86.3)
- added J2: BOOT, Connector_PinHeader_2.54mm:PinHeader_1x02_P2.54mm_Vertical, F.Cu at (174.0, 52.4)
- added J2: BOOT, Connector_PinHeader_2.54mm:PinHeader_1x02_P2.54mm_Vertical, F.Cu at (124.0, 52.4)
- added R1: 10k, Resistor_SMD:R_0603_1608Metric, F.Cu at (172.4, 93.2)
- added R1: 10k, Resistor_SMD:R_0603_1608Metric, F.Cu at (122.4, 93.2)
- added R1: 10k, Resistor_SMD:R_0603_1608Metric, F.Cu at (172.4, 59.2)
- added R10: 1k, Resistor_SMD:R_0603_1608Metric, F.Cu at (178.1, 111.0)
- added R10: 1k, Resistor_SMD:R_0603_1608Metric, F.Cu at (128.1, 111.0)
- added R10: 1k, Resistor_SMD:R_0603_1608Metric, F.Cu at (178.1, 77.0)
- added R11: 0, Resistor_SMD:R_0603_1608Metric, B.Cu at (172.5, 110.0)
- added R11: 0, Resistor_SMD:R_0603_1608Metric, B.Cu at (122.5, 110.0)
- added R11: 0, Resistor_SMD:R_0603_1608Metric, B.Cu at (172.5, 76.0)
- added R12: 0, Resistor_SMD:R_0603_1608Metric, B.Cu at (174.1, 98.8)
- added R12: 0, Resistor_SMD:R_0603_1608Metric, B.Cu at (124.1, 98.8)
- added R12: 0, Resistor_SMD:R_0603_1608Metric, B.Cu at (174.1, 64.8)
- added R12: 0, Resistor_SMD:R_0603_1608Metric, B.Cu at (124.1, 64.8)
- added R13: 0, Resistor_SMD:R_0603_1608Metric, B.Cu at (172.5, 105.9)
- added R13: 0, Resistor_SMD:R_0603_1608Metric, B.Cu at (122.5, 105.9)
- added R13: 0, Resistor_SMD:R_0603_1608Metric, B.Cu at (172.5, 71.9)
- added R13: 0, Resistor_SMD:R_0603_1608Metric, B.Cu at (122.5, 71.9)
- added R14: 0, Resistor_SMD:R_0603_1608Metric, B.Cu at (172.6, 92.8)
- added R14: 0, Resistor_SMD:R_0603_1608Metric, B.Cu at (122.6, 92.8)
- added R14: 0, Resistor_SMD:R_0603_1608Metric, B.Cu at (172.6, 58.8)
- added R15: 0, Resistor_SMD:R_0603_1608Metric, B.Cu at (172.5, 108.0)
- added R15: 0, Resistor_SMD:R_0603_1608Metric, B.Cu at (122.5, 108.0)
- added R15: 0, Resistor_SMD:R_0603_1608Metric, B.Cu at (172.5, 74.0)
- added R16: 0, Resistor_SMD:R_0603_1608Metric, B.Cu at (171.1, 92.8)
- added R16: 0, Resistor_SMD:R_0603_1608Metric, B.Cu at (121.1, 92.8)
- added R16: 0, Resistor_SMD:R_0603_1608Metric, B.Cu at (171.1, 58.8)
- added R2: 10k, Resistor_SMD:R_0603_1608Metric, B.Cu at (168.8, 87.2)
- added R2: 10k, Resistor_SMD:R_0603_1608Metric, B.Cu at (118.8, 87.2)
- added R2: 10k, Resistor_SMD:R_0603_1608Metric, B.Cu at (168.8, 53.2)
- added R3: 5.1k, Resistor_SMD:R_0603_1608Metric, B.Cu at (158.1, 97.4)
- added R3: 5.1k, Resistor_SMD:R_0603_1608Metric, B.Cu at (108.1, 97.4)
- added R3: 5.1k, Resistor_SMD:R_0603_1608Metric, B.Cu at (158.1, 63.4)
- added R5: 27, Resistor_SMD:R_0603_1608Metric, B.Cu at (160.3, 101.3)
- added R5: 27, Resistor_SMD:R_0603_1608Metric, B.Cu at (110.3, 101.3)
- added R5: 27, Resistor_SMD:R_0603_1608Metric, B.Cu at (160.3, 67.3)
- added R6: 27, Resistor_SMD:R_0603_1608Metric, B.Cu at (160.3, 99.8)
- added R6: 27, Resistor_SMD:R_0603_1608Metric, B.Cu at (110.3, 99.8)
- added R6: 27, Resistor_SMD:R_0603_1608Metric, B.Cu at (160.3, 65.8)
- added R7: 1k, Resistor_SMD:R_0603_1608Metric, F.Cu at (178.1, 112.5)
- added R7: 1k, Resistor_SMD:R_0603_1608Metric, F.Cu at (128.1, 112.5)
- added R7: 1k, Resistor_SMD:R_0603_1608Metric, F.Cu at (178.1, 78.5)
- added R8: 100k, Resistor_SMD:R_0603_1608Metric, B.Cu at (177.9, 102.8)
- added R8: 100k, Resistor_SMD:R_0603_1608Metric, B.Cu at (127.9, 102.8)
- added R8: 100k, Resistor_SMD:R_0603_1608Metric, B.Cu at (177.9, 68.8)
- added R8: 100k, Resistor_SMD:R_0603_1608Metric, B.Cu at (127.9, 68.8)
- added R9: 0, Resistor_SMD:R_0603_1608Metric, B.Cu at (169.6, 92.8)
- added R9: 0, Resistor_SMD:R_0603_1608Metric, B.Cu at (119.6, 92.8)
- added R9: 0, Resistor_SMD:R_0603_1608Metric, B.Cu at (169.6, 58.8)
- added TP10: TestPoint, TestPoint:TestPoint_Pad_D1.0mm, B.Cu at (153.7, 92.8)
- added TP10: TestPoint, TestPoint:TestPoint_Pad_D1.0mm, B.Cu at (103.7, 92.8)
- added TP10: TestPoint, TestPoint:TestPoint_Pad_D1.0mm, B.Cu at (153.7, 58.8)
- added TP10: TestPoint, TestPoint:TestPoint_Pad_D1.0mm, B.Cu at (103.7, 58.8)
- added TP8: TestPoint, TestPoint:TestPoint_Pad_D1.0mm, B.Cu at (165.8, 93.3)
- added TP8: TestPoint, TestPoint:TestPoint_Pad_D1.0mm, B.Cu at (115.8, 93.3)
- added TP8: TestPoint, TestPoint:TestPoint_Pad_D1.0mm, B.Cu at (165.8, 59.3)
- added TP8: TestPoint, TestPoint:TestPoint_Pad_D1.0mm, B.Cu at (115.8, 59.3)
- added TP9: TestPoint, TestPoint:TestPoint_Pad_D1.0mm, B.Cu at (167.6, 92.4)
- added TP9: TestPoint, TestPoint:TestPoint_Pad_D1.0mm, B.Cu at (117.6, 92.4)
- added TP9: TestPoint, TestPoint:TestPoint_Pad_D1.0mm, B.Cu at (167.6, 58.4)
- added TP9: TestPoint, TestPoint:TestPoint_Pad_D1.0mm, B.Cu at (117.6, 58.4)
- added U1: SIT2001B, Package_TO_SOT_SMD:SOT-23-5, B.Cu at (174.6, 96.2)
- added U1: SIT2001B, Package_TO_SOT_SMD:SOT-23-5, B.Cu at (124.6, 96.2)
- added U1: SIT2001B, Package_TO_SOT_SMD:SOT-23-5, B.Cu at (174.6, 62.2)
- added U1: SIT2001B, Package_TO_SOT_SMD:SOT-23-5, B.Cu at (124.6, 62.2)
- added U3: RP2040, rp2040:RP2040_QFN56_HandSolderHack, B.Cu at (168.4, 99.4)
- added U3: RP2040, rp2040:RP2040_QFN56_HandSolderHack, B.Cu at (118.4, 99.4)
- added U3: RP2040, rp2040:RP2040_QFN56_HandSolderHack, B.Cu at (168.4, 65.4)
- C11, C6, C8, C9: moved to F.Cu
- L1 (x4): value 600R/0.5A/N.F. -> N.F.
- L2 (x4): value 600R/0.5A -> N.F.
- R2: moved to B.Cu
- U3: footprint Package_DFN_QFN:QFN-56-1EP_7x7mm_P0.4mm_EP5.6x5.6mm -> rp2040:RP2040_QFN56_HandSolderHack
- moved R1 6.45 mm to (122.4, 59.2), turned to 90 degrees
- moved R2 6.40 mm to (118.8, 53.2), turned to 270 degrees
- moved R9 5.56 mm to (119.6, 58.8), turned to 90 degrees
- moved C8 5.04 mm to (115.0, 64.7), turned to 270 degrees
- moved C2 4.48 mm to (124.9, 59.6), turned to 180 degrees
- moved R10 3.50 mm to (128.1, 77.0), turned to 0 degrees
- moved R16 3.41 mm to (121.1, 58.8), turned to 90 degrees
- moved C9 3.17 mm to (113.5, 64.7), turned to 270 degrees
- moved D4 3.07 mm to (131.1, 77.0), turned to 180 degrees
- moved R15 2.72 mm to (122.5, 74.0)
- moved R11 2.70 mm to (122.5, 76.0)
- moved R7 2.49 mm to (128.1, 78.5), turned to 0 degrees
- moved C11 1.98 mm to (116.1, 69.8), turned to 90 degrees
- moved C6 1.97 mm to (114.1, 69.8), turned to 90 degrees
- moved R14 1.97 mm to (122.6, 58.8), turned to 90 degrees
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Connections:
- J4 pad 11: Net-(J4-Pad11) -> (no net) (x4)
- R7 pad 1: +3V3 -> /VO
- U3 pad 24: /SWCLK -> (no net)
- U3 pad 25: /SWDIO -> (no net)
- U3 pad 26: /RUN -> Net-(C7-Pad1)
- U3 pad 30: /RTCK -> /TDO_SWO
- U3 pad 31: /TDO_SWO -> /~SRST
- U3 pad 32: /~SRST -> (no net)
Routing:
- net GND: track 490.2 -> 1305.2 mm, vias 676 -> 624
- net +3V3: track 576.8 -> 393.6 mm, vias 40 -> 48
- net /SWCLK: track 60.7 -> 0.00 mm
- net Net-(J4-Pad11): track 50.7 -> 0.00 mm
- net +1V1: track 216.4 -> 262.4 mm
- net /UART_TX: track 60.1 -> 16.2 mm
- net /UART_RX: track 51.7 -> 11.6 mm
- net Net-(J4-Pad3): track 51.7 -> 90.4 mm
- net /SWDIO: track 38.5 -> 0.00 mm
- net /LED: track 97.6 -> 67.2 mm
- net Net-(J4-Pad5): track 52.9 -> 80.2 mm
- net /RTCK: track 26.6 -> 0.00 mm
- net Net-(C7-Pad1): track 0.00 -> 25.8 mm
- net /RUN: track 24.6 -> 0.00 mm, vias 4 -> 0
- net /~TRST: track 32.6 -> 9.97 mm
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- added copper zone on F.Cu, net /D+
- added copper zone on F.Cu, net /D-
- added copper zone on B.Cu, net /QSPI_CSN
- removed copper zone on F.Cu, net +3V3
- removed copper zone on F.Cu, net /VBUS
Other:
- board size 103.1 x 81.2 mm -> 109.1 x 77.8 mm
- board text added: "RP2040 CMSIS-DAP version 2022/06/01 @tnishinaga"
- board text removed: "3v3"
- board text removed: "BOOT"
- board text removed: "CLK"
- board text removed: "DIO"
- board text removed: "G"
- board text removed: "GND"
- board text removed: "RP2040 CMSIS-DAP version 2022/04/09 @tnishinaga"
- board text removed: "RUN"
- board text removed: "RX<"
- board text removed: "SWD"
- board text removed: "TX>"
